Commit message: correct for x-axis forward in rectract position

File: urdf/chris_kinova_lab.xacro (robot description, xacro)
@@ -75,5 +75,5 @@
     <parent link="base_plate" />
     <child link="kinova_mount_post" />
-    <origin xyz="0 0 0.036" rpy="0 0 0" />
+    <origin xyz="0 0 0.036" rpy="0 0 ${M_PI/2}" />
   </joint>
   <xacro:property name="robot_root" value="kinova_mount_post" />
@@ -81,5 +81,5 @@
   <joint name="kinect_base_joint" type="fixed">
     <axis xyz="0 0 1" />
-    <origin xyz="-0.0508 0.2286 0.035" rpy="0 0 -0.1745"/>
+    <origin xyz="-0.0508 0.2286 0.035" rpy="0 0 ${-0.174533}"/>
     <parent link="base_plate"/>
     <child link="camera_link"/>
@@ -88,5 +88,5 @@
   <joint name="hokuyo_base_joint" type="fixed">
     <axis xyz="0 0 1" />
-    <origin xyz="-0.073 -0.2286 0.019" rpy="0 0 0.1745"/>
+    <origin xyz="-0.073 -0.2286 0.019" rpy="0 0 ${0.174533}"/>
     <parent link="base_plate"/>
     <child link="hokuyo_base_link"/>

Commit message: lab setup with moveit

File: urdf/chris_kinova_lab.xacro (robot description, xacro)
@@ -48,5 +48,5 @@
     <material>Gazebo/DarkGrey</material>
   </gazebo>
-  <link name="kinova_mount_post">
+  <link name="root">
     <visual>
       <origin xyz="0 0 -0.0104" rpy="0 0 0" />
@@ -57,5 +57,5 @@
     </visual>
   </link>
-  <gazebo reference="kinova_mount_post">
+  <gazebo reference="root">
     <material>Gazebo/DarkGrey</material>
   </gazebo>
@@ -74,8 +74,8 @@
   <joint name="connect_base_and_mount_post" type="fixed">
     <parent link="base_plate" />
-    <child link="kinova_mount_post" />
+    <child link="root" />
     <origin xyz="0 0 0.036" rpy="0 0 ${M_PI/2}" />
   </joint>
-  <xacro:property name="robot_root" value="kinova_mount_post" />
+  <xacro:property name="robot_root" value="root" />
   <xacro:m1n6s200  base_parent="${robot_root}" use_ring_mesh="true" />
   <joint name="kinect_base_joint" type="fixed">

Commit message: move sensor positions; simulation used same topic has H/W for point clouds

File: urdf/chris_kinova_lab.xacro (robot description, xacro)
@@ -81,5 +81,5 @@
   <joint name="kinect_base_joint" type="fixed">
     <axis xyz="0 0 1" />
-    <origin xyz="-0.0508 0.2286 0.035" rpy="0 0 ${-0.174533}"/>
+    <origin xyz="-0.30 0.25 0.016" rpy="0 -0.05 -0.174533"/>
     <parent link="base_plate"/>
     <child link="camera_link"/>
@@ -88,5 +88,5 @@
   <joint name="hokuyo_base_joint" type="fixed">
     <axis xyz="0 0 1" />
-    <origin xyz="-0.073 -0.2286 0.019" rpy="0 0 ${0.174533}"/>
+    <origin xyz="0.105 0.0 0.019" rpy="0 0 0"/>
     <parent link="base_plate"/>
     <child link="hokuyo_base_link"/>

File: urdf/sensors/kinect_gazebo.urdf.xacro (robot description, xacro)
@@ -25,5 +25,5 @@
           <imageTopicName>rgb/image_raw</imageTopicName>
           <depthImageTopicName>depth/image_raw</depthImageTopicName>
-          <pointCloudTopicName>depth/points</pointCloudTopicName>
+          <pointCloudTopicName>depth_registered/points</pointCloudTopicName>
           <cameraInfoTopicName>rgb/camera_info</cameraInfoTopicName>
           <depthImageCameraInfoTopicName>depth/camera_info</depthImageCameraInfoTopicName>

Commit message: remove material properties that  would not load; remove --inorder; add collision geometry

File: urdf/chris_kinova_lab.xacro (robot description, xacro)
@@ -24,12 +24,12 @@
         <box size = "0.4064 0.762 0.01905"/>
       </geometry>
-      <material name="material_blue" />
+      <!-- material name="material_blue" / -->
     </visual>
-    <!--collision>
-      <origin xyz="0 0 0" rpy="0 0 0" />
+    <collision>
+      <origin xyz="0 0 -0.009525" rpy="0 0 0" />
       <geometry>
-        <box size = "0.25 0.25 0.02"/>
+        <box size = "0.4064 0.762 0.01905"/>
       </geometry>
-    </collision-->
+    </collision>
   </link>
   <gazebo reference="base_plate">
@@ -42,6 +42,12 @@
         <box size = "0.1461 0.1981 0.01905"/>
       </geometry>
-      <material name="material_dark_grey" />
+      <!-- material name="material_dark_grey" / -->
     </visual>
+    <collision>
+      <origin xyz="0 0 0.009525" rpy="0 0 0" />
+      <geometry>
+        <box size = "0.1461 0.1981 0.01905"/>
+      </geometry>
+    </collision>
   </link>
   <gazebo reference="kinova_mount_base">
@@ -54,6 +60,13 @@
         <box size = "0.03 0.03 0.0608"/>
       </geometry>
-      <material name="material_dark_grey" />
+      <!-- material name="material_dark_grey" /-->
     </visual>
+    <collision>
+      <origin xyz="0 0 -0.0104" rpy="0 0 0" />
+      <geometry>
+        <box size = "0.03 0.03 0.0608"/>
+      </geometry>
+      <!-- material name="material_dark_grey" /-->
+    </collision>
   </link>
   <gazebo reference="root">
@@ -85,5 +98,5 @@
     <child link="camera_link"/>
   </joint>
-  <sensor_kinect  parent="base_plate"/>
+  <xacro:sensor_kinect  parent="base_plate"/>
   <joint name="hokuyo_base_joint" type="fixed">
     <axis xyz="0 0 1" />

File: urdf/sensors/hokuyo_urg04.urdf.xacro (robot description, xacro)
@@ -52,5 +52,5 @@
   </link>
   <!-- Simulation sensors -->
-  <hokuyo_urg04_sim/>
+  <xacro:hokuyo_urg04_sim/>
   </xacro:macro>
 </robot>

File: urdf/sensors/kinect.urdf.xacro (robot description, xacro)
@@ -58,5 +58,5 @@
 	<link name="camera_depth_optical_frame"/>
 	<!-- Kinect sensor for simulation -->
-	<kinect_sim_3dsensor/>
+	<xacro:kinect_sim_3dsensor/>
   </xacro:macro>
 </robot>
