Commit message: update setup for ros2 controllers and compatability with new chris_kinova_driver

File: urdf/kinova.ros2_control.xacro (robot description, xacro)
@@ -1,5 +1,5 @@
 <?xml version="1.0"?>
 <root xmlns:xacro="http://www.ros.org/wiki/xacro">
-<xacro:macro name="gazebo_config" params="robot_namespace
+<xacro:macro name="ros2_control_config" params="robot_namespace
                 prefix
                 use_mock_hardware:=^|false
@@ -18,5 +18,5 @@
         </xacro:if>
         <xacro:unless value="${use_mock_hardware or sim_gazebo}">
-          <plugin>chris_kinova_hardware/KinovaHardwareInterface</plugin>
+          <plugin>chris_kinova_driver/KinovaMicoInterfaceHardware</plugin>
         </xacro:unless>
       </hardware>
@@ -24,4 +24,5 @@
         <command_interface name="position" />
         <command_interface name="velocity" />
+        <command_interface name="effort" />
         <state_interface name="position">
           <param name="initial_value">0.0</param>
@@ -30,8 +31,12 @@
           <param name="initial_value">0.0</param>
         </state_interface>
+        <state_interface name="effort">
+          <param name="initial_value">0.0</param>
+        </state_interface>
       </joint>
       <joint name="${prefix}_joint_2">
         <command_interface name="position" />
         <command_interface name="velocity" />
+        <command_interface name="effort" />
         <state_interface name="position">
           <param name="initial_value">${300/180*J_PI}</param>
@@ -40,8 +45,12 @@
           <param name="initial_value">0.0</param>
         </state_interface>
+        <state_interface name="effort">
+          <param name="initial_value">0.0</param>
+        </state_interface>
       </joint>
       <joint name="${prefix}_joint_3">
         <command_interface name="position" />
         <command_interface name="velocity" />
+        <command_interface name="effort" />
         <state_interface name="position">
           <param name="initial_value">${300/180*J_PI}</param>
@@ -50,8 +59,12 @@
           <param name="initial_value">0.0</param>
         </state_interface>
+        <state_interface name="effort">
+          <param name="initial_value">0.0</param>
+        </state_interface>
       </joint>
       <joint name="${prefix}_joint_4">
         <command_interface name="position" />
         <command_interface name="velocity" />
+        <command_interface name="effort" />
         <state_interface name="position">
           <param name="initial_value">0.0</param>
@@ -60,8 +73,12 @@
           <param name="initial_value">0.0</param>
         </state_interface>
+        <state_interface name="effort">
+          <param name="initial_value">0.0</param>
+        </state_interface>
       </joint>
       <joint name="${prefix}_joint_5">
         <command_interface name="position" />
         <command_interface name="velocity" />
+        <command_interface name="effort" />
         <state_interface name="position">
           <param name="initial_value">0.0</param>
@@ -70,8 +87,12 @@
           <param name="initial_value">0.0</param>
         </state_interface>
+        <state_interface name="effort">
+          <param name="initial_value">0.0</param>
+        </state_interface>
       </joint>
       <joint name="${prefix}_joint_6">
         <command_interface name="position" />
         <command_interface name="velocity" />
+        <command_interface name="effort" />
         <state_interface name="position">
           <param name="initial_value">0.0</param>
@@ -80,8 +101,12 @@
           <param name="initial_value">0.0</param>
         </state_interface>
+        <state_interface name="effort">
+          <param name="initial_value">0.0</param>
+        </state_interface>
       </joint>
       <joint name="${prefix}_joint_finger_1">
         <command_interface name="position" />
         <command_interface name="velocity" />
+        <command_interface name="effort" />
         <state_interface name="position">
           <param name="initial_value">0.0</param>
@@ -90,12 +115,19 @@
           <param name="initial_value">0.0</param>
         </state_interface>
+        <state_interface name="effort">
+          <param name="initial_value">0.0</param>
+        </state_interface>
       </joint>
       <joint name="${prefix}_joint_finger_2">
         <command_interface name="position" />
         <command_interface name="velocity" />
+        <command_interface name="effort" />
         <state_interface name="position">
           <param name="initial_value">0.0</param>
         </state_interface>
         <state_interface name="velocity">
+          <param name="initial_value">0.0</param>
+        </state_interface>
+        <state_interface name="effort">
           <param name="initial_value">0.0</param>
         </state_interface>

File: urdf/m1n6s200.urdf.xacro (robot description, xacro)
@@ -21,5 +21,5 @@
     <xacro:include filename="$(find chris_kinova_bringup)/urdf/kinova_finger_set.xacro" />
     <!-- Import all Gazebo-customization elements -->
-    <xacro:include filename="$(find chris_kinova_bringup)/urdf/kinova.gazebo" />
+    <xacro:include filename="$(find chris_kinova_bringup)/urdf/kinova.ros2_control.xacro" />
     <xacro:property name="link_base_mesh" value="base" />
     <xacro:property name="link_1_mesh" value="shoulder" />
@@ -113,5 +113,6 @@
                 sim_gazebo:=^|false"
                >
-        <xacro:gazebo_config robot_namespace="${prefix}"
+        <!-- set up ros2 control and gazebo sim interfaces -->
+        <xacro:ros2_control_config robot_namespace="${prefix}"
                 use_mock_hardware="$(arg use_mock_hardware)"
                 mock_sensor_commands="$(arg mock_sensor_commands)"
